File: 2.Device Hardware/_autosave-Abhoinn_IoT_V2.kicad_pcb (KiCad board)
At the start: 4 copper layers, 96 x 96 mm, 46 parts, among them IC1 AX-SIP-SFEU-1-01-TX30, IC2 MS5840-02BA01, J1 Conn_01x02, J2 Conn_01x02, J3 Conn_02x05_Odd_Even, J4 Conn_02x05_Odd_Even, J5 Conn_Coaxial, J6 Conn_01x02_Female, P1 USB_C_Plug_USB2.0, U1 XC6206PxxxMR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

Commit message: PCB updates
Parts:
- moved J5 1.38 mm to (121.6, 79.3)
Routing:
- net GND: track 30.7 -> 64.9 mm, vias 16 -> 36
- net Net-(P1-PadS1): track 0.00 -> 30.1 mm
- net +5V: track 54.5 -> 70.1 mm
- net Net-(P1-PadA4): track 0.00 -> 5.96 mm
- net Net-(IC1-Pad3): track 10.1 -> 8.60 mm
- added copper zone on In2.Cu, net +3V3
- added copper zone on In1.Cu, net GND

Commit message: update PCB
Routing:
- net GND: track 64.9 -> 65.7 mm, vias 36 -> 61
- net +3V3: vias 9 -> 17
Other:
- board text added: "Abhainn IoT V2"
- board text added: "Abhainn-IoT Hardware Components by Cian Vaugh is licensed under a Creative Commons Attribution-NonCommercial-ShareAlike 4.0 International License."
