File: 2.Device Hardware/_autosave-Abhoinn_IoT_V2.kicad_pcb (KiCad board)
At the start: 4 copper layers, 96 x 96 mm, 46 parts, among them IC1 AX-SIP-SFEU-1-01-TX30, IC2 MS5840-02BA01, J1 Conn_01x02, J2 Conn_01x02, J3 Conn_02x05_Odd_Even, J4 Conn_02x05_Odd_Even, J5 Conn_Coaxial, J6 Conn_01x02_Female, P1 USB_C_Plug_USB2.0, U1 XC6206PxxxMR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

Commit message: update
Connections:
- F1 pad 2: Net-(D1-Pad1) -> Net-(F1-Pad2)
- FB1 pad 1: Net-(D1-Pad1) -> Net-(F1-Pad2)
Routing:
- net Net-(D4-Pad2): track 8.10 -> 34.5 mm
- net Net-(F1-Pad2): track 0.00 -> 5.06 mm
- net Net-(D1-Pad1): track 10.1 -> 5.08 mm
- net +3V3: track 44.8 -> 42.0 mm, vias 9 -> 23
- net GND: track 64.9 -> 65.8 mm, vias 36 -> 63
- net PRESSURE_SCL: track 15.8 -> 16.5 mm
Other:
- board outline removed

Commit message: v2 final and production files
Routing:
- net +3V3: track 42.0 -> 43.5 mm, vias 23 -> 26
- net GND: vias 63 -> 80
Other:
- board outline added: 96 x 96 mm
