File: 2.Device Hardware/Abhoinn_IoT_V3.sch (KiCad schematic (older format))
At the start: 46 parts, among them IC1 AX-SIP-SFEU-1-01-TX30, IC2 MS5840-02BA01, J1 Conn_01x02, J2 Conn_01x02, J3 Conn_02x05_Odd_Even, J4 Conn_02x05_Odd_Even, J5 Conn_Coaxial, J6 Conn_01x02_Female, P1 USB_C_Plug_USB2.0, U1 XC6206PxxxMR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

Commit message: updates
Parts:
- removed P1: USB_C_Plug_USB2.0, Connector_USB:USB_C_Receptacle_Amphenol_12401548E4-2A, symbol Connector:USB_C_Plug_USB2.0
- removed R9: 56k, Resistor_SMD:R_0603_1608Metric_Pad0.98x0.95mm_HandSolder, symbol Device:R_Small
- removed U2: USBLC6-2SC6, Package_TO_SOT_SMD:SOT-23-6, symbol Power_Protection:USBLC6-2SC6
- D1: footprint Diode_SMD:D_SMA-SMB_Universal_Handsoldering -> Diode_SMD:D_SMA_Handsoldering
- F1: footprint Fuse:Fuse_2010_5025Metric_Pad1.52x2.65mm_HandSolder -> Fuse:Fuse_1206_3216Metric_Pad1.42x1.75mm_HandSolder
- J1, J2: footprint Connector_PinSocket_2.00mm:PinSocket_1x02_P2.00mm_Vertical -> Connector_PinSocket_2.54mm:PinSocket_1x02_P2.54mm_Vertical
- J3, J4: footprint Connector_PinSocket_2.00mm:PinSocket_2x05_P2.00mm_Vertical -> Connector_PinSocket_2.54mm:PinSocket_2x05_P2.54mm_Vertical
- JP1, JP2, JP3, JP4: footprint Connector_PinSocket_2.00mm:PinSocket_1x03_P2.00mm_Vertical -> Connector_PinSocket_2.54mm:PinSocket_1x03_P2.54mm_Vertical
Connections:
- net labels removed: D+, D-, USB_D+, USB_D-
- wire segments 110 -> 105
Other:
- note removed: "Shield grounded on hoast sided\n"
- note removed: "USB data + and - roughted as differntal pare"
- moved on the sheet: C9, IC2, R5
