File: 2.Device Hardware/Abhionn-IoT_v3/Abhoinn_IoT_V3.kicad_pcb (KiCad board)
At the start: 4 copper layers, 60 x 50 mm, 43 parts, among them IC1 AX-SIP-SFEU-1-01-TX30, IC2 MS5840-02BA01, J1 Conn_01x02, J2 Conn_01x02, J3 Conn_02x05_Odd_Even, J4 Conn_02x05_Odd_Even, J5 Conn_Coaxial, J6 Conn_01x02_Female, U1 XC6206PxxxMR, U3 STM32L082KZTx

Commit message: Formating
Other:
- net class Default removed
- net class Min 1oz removed
- net class POWER+ removed
- net class RF removed
